File: Arduino/board_lock-ponto.brd (EAGLE design)
At the start: 4 parts

Commit message: Preparing to add token
Parts:
- E$1: device SHIELD-LCD16x2_Rev_B:ARDUINO_SH_LCD-PLATFORM -> converter_lcd_serial_i2c:LCD-I2C-CONVERTER
- E$3: device converter_lcd_serial_i2c:LCD-I2C-CONVERTER -> display-lcd:TUXGR_16X2_R2
- moved E$3 90.6 mm to (74.9, 80.0), flipped to the top, turned to 0 degrees
- moved E$1 90.3 mm to (62.2, 111.2), flipped to the bottom, turned to 180 degrees
- moved E$2 26.0 mm to (50.8, 38.1)
- moved E$4 15.5 mm to (41.5, 38.0)
Connections:
- new net S$18: E$2.SCK, E$4.7
- new net S$19: E$2.MOSI, E$4.6
- new net S$20: E$2.MISO, E$4.5
- new net S$21: E$2.IRQ, E$4.4
- new net S$22: E$2.GND, E$4.3
- new net S$23: E$2.RST, E$4.2
- new net S$24: E$2.3V3, E$4.1
- net S$1: now also E$1.J2.16, E$3.1; no longer E$1.D10, E$3.J2.1
- net S$10: now also E$1.J2.7, E$3.10; no longer E$2.SS, E$4.8
- net S$11: now also E$1.J2.6, E$3.11; no longer E$2.SCK, E$4.7
- net S$12: now also E$1.J2.4, E$3.13; no longer E$2.MOSI, E$4.6
- net S$13: now also E$1.J2.3, E$3.14; no longer E$2.MISO, E$4.5
- net S$14: now also E$1.J2.2, E$3.15; no longer E$2.IRQ, E$4.4
- net S$15: now also E$1.J2.1, E$3.16; no longer E$2.3V3, E$4.1
- net S$16: now also E$1.J2.5, E$3.12; no longer E$2.RST, E$4.2
- net S$17: now also E$2.SS, E$4.8; no longer E$2.GND, E$4.3
- net S$2: now also E$1.J2.15, E$3.2; no longer E$1.D9, E$3.J2.11
- net S$3: now also E$1.J2.14, E$3.3; no longer E$1.D8, E$3.J2.13
- net S$4: now also E$1.J2.13, E$3.4; no longer E$1.D7, E$3.J2.3
- net S$5: now also E$1.J2.12, E$3.5; no longer E$1.D6, E$3.J2.4
- net S$6: now also E$1.J2.11, E$3.6; no longer E$1.D5, E$3.J2.5
- net S$7: now also E$1.J2.10, E$3.7; no longer E$1.D4, E$3.J2.6
- net S$8: now also E$1.J2.9, E$3.8; no longer E$1.GND, E$3.J2.16
- net S$9: now also E$1.J2.8, E$3.9; no longer E$1.5V, E$3.J2.15
Routing:
- net S$3: track 236.5 -> 9.46 mm
- net S$2: track 125.6 -> 9.46 mm
- net S$7: track 94.4 -> 9.46 mm
- net S$6: track 89.3 -> 9.46 mm
- net S$5: track 84.6 -> 9.46 mm
- net S$8: track 83.7 -> 9.46 mm
- net S$4: track 79.8 -> 9.46 mm
- net S$9: track 72.7 -> 9.46 mm
- net S$1: track 71.0 -> 9.46 mm
- net S$19: track 0.00 -> 10.6 mm
- net S$21: track 0.00 -> 10.3 mm
- net S$22: track 0.00 -> 10.1 mm
- net S$23: track 0.00 -> 10.1 mm
- net S$18: track 0.00 -> 10.1 mm
- net S$24: track 0.00 -> 10.0 mm
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