File: Arduino/lock_board.brd (EAGLE design)
At the start: 80 x 53.3 mm, 3 parts

Commit message: Preparing to add token
Parts:
- added E$4: (no value), con-lsta:FE08
- moved E$2 7.50 mm to (30.0, 15.0)
Connections:
- new net S$10: E$2.SS, E$4.8
- new net S$11: E$2.SCK, E$4.7
- new net S$12: E$2.MOSI, E$4.6
- new net S$13: E$2.MISO, E$4.5
- new net S$14: E$2.IRQ, E$4.4
- new net S$15: E$2.3V3, E$4.1
- new net S$16: E$2.RST, E$4.2
- new net S$17: E$2.GND, E$4.3
Routing:
- net S$3: track 225.9 -> 236.5 mm
- net S$8: track 74.9 -> 83.7 mm
- net S$9: track 64.8 -> 72.7 mm
- net S$15: track 0.00 -> 7.61 mm
- net S$17: track 0.00 -> 7.50 mm
- net S$16: track 0.00 -> 7.50 mm
- net S$14: track 0.00 -> 7.50 mm
- net S$13: track 0.00 -> 7.50 mm
- net S$12: track 0.00 -> 7.50 mm
- net S$11: track 0.00 -> 7.50 mm
- net S$10: track 0.00 -> 7.50 mm
Other:
- board outline removed
Changed lines of the file:
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@@
 <?xml version="1.0" encoding="utf-8"?>
 <!DOCTYPE eagle SYSTEM "eagle.dtd">
-<eagle version="7.6.0">
+<eagle version="8.2.2">
 <drawing>
 <settings>
@@
 <layers>
 <layer number="1" name="Top" color="4" fill="1" visible="yes" active="yes"/>
+<layer number="2" name="Route2" color="1" fill="3" visible="no" active="no"/>
+<layer number="3" name="Route3" color="4" fill="3" visible="no" active="no"/>
+<layer number="4" name="Route4" color="1" fill="4" visible="no" active="no"/>
+<layer number="5" name="Route5" color="4" fill="4" visible="no" active="no"/>
+<layer number="6" name="Route6" color="1" fill="8" visible="no" active="no"/>
+<layer number="7" name="Route7" color="4" fill="8" visible="no" active="no"/>
+<layer number="8" name="Route8" color="1" fill="2" visible="no" active="no"/>
+<layer number="9" name="Route9" color="4" fill="2" visible="no" active="no"/>
+<layer number="10" name="Route10" color="1" fill="7" visible="no" active="no"/>
+<layer number="11" name="Route11" color="4" fill="7" visible="no" active="no"/>
+<layer number="12" name="Route12" color="1" fill="5" visible="no" active="no"/>
+<layer number="13" name="Route13" color="4" fill="5" visible="no" active="no"/>
+<layer number="14" name="Route14" color="1" fill="6" visible="no" active="no"/>
+<layer number="15" name="Route15" color="4" fill="6" visible="no" active="no"/>
 <layer number="16" name="Bottom" color="1" fill="1" visible="no" active="yes"/>
 <layer number="17" name="Pads" color="2" fill="1" visible="yes" active="yes"/>
@@
 <elements>
 <element name="E$1" library="SHIELD-LCD16x2_Rev_B" package="ARDUINO_SH_LCD-PLATFORM" value="" x="2.55" y="43.51"/>
-<element name="E$2" library="mfrc522-module" package="RFID-RC522" value="" x="30" y="22.5" rot="R90"/>
+<element name="E$2" library="mfrc522-module" package="RFID-RC522" value="" x="30" y="15" rot="R90"/>
 <element name="E$3" library="converter_lcd_serial_i2c" package="LCD-I2C-CONVERTER" value="" x="7.5" y="19.5" rot="MR90"/>
+<element name="E$4" library="con-lsta" package="FE08" value="" x="22.5" y="15" rot="R90"/>
 </elements>
 <signals>
@@
 <wire x1="5.07" y1="8.07" x2="-1.5" y2="1.5" width="1.27" layer="1"/>
 <wire x1="-1.5" y1="1.5" x2="-1.5" y2="-1.5" width="1.27" layer="1"/>
-<wire x1="-1.5" y1="-1.5" x2="1.5" y2="-4.5" width="1.27" layer="1"/>
-<wire x1="1.5" y1="-4.5" x2="13.5" y2="-4.5" width="1.27" layer="1"/>
-<wire x1="13.5" y1="-4.5" x2="15" y2="-6" width="1.27" layer="1"/>
-<wire x1="15" y1="-6" x2="31.5" y2="-6" width="1.27" layer="1"/>
-<wire x1="31.5" y1="-6" x2="63" y2="25.5" width="1.27" layer="1"/>
-<wire x1="63" y1="25.5" x2="63" y2="34.5" width="1.27" layer="1"/>
-<wire x1="63" y1="34.5" x2="67.5" y2="39" width="1.27" layer="1"/>
-<wire x1="67.5" y1="39" x2="76.5" y2="39" width="1.27" layer="1"/>
-<wire x1="76.5" y1="39" x2="82.5" y2="45" width="1.27" layer="1"/>
-<wire x1="82.5" y1="45" x2="82.5" y2="48" width="1.27" layer="1"/>
-<wire x1="82.5" y1="48" x2="72" y2="58.5" width="1.27" layer="1"/>
+<wire x1="-0.374746875" y1="-2.625253125" x2="-1.5" y2="-1.5" width="1.27" layer="1"/>
+<wire x1="-0.374746875" y1="-2.625253125" x2="1.5" y2="-4.5" width="1.27" layer="1"/>
+<wire x1="72" y1="58.5" x2="82.5" y2="48" width="1.27" layer="1"/>
 <wire x1="72" y1="58.5" x2="72" y2="85.5" width="1.27" layer="1"/>
 <wire x1="72" y1="85.5" x2="75" y2="88.5" width="1.27" layer="1"/>
@@
 <wire x1="55.636" y1="94.636" x2="60" y2="99" width="1.27" layer="1"/>
 <wire x1="60" y1="99" x2="79.5" y2="99" width="1.27" layer="1"/>
+<wire x1="82.5" y1="43.5" x2="79.5" y2="40.5" width="1.27" layer="1"/>
+<wire x1="79.5" y1="40.5" x2="66" y2="40.5" width="1.27" layer="1"/>
+<wire x1="66" y1="40.5" x2="63" y2="37.5" width="1.27" layer="1"/>
+<wire x1="63" y1="37.5" x2="63" y2="12" width="1.27" layer="1"/>
+<wire x1="45" y1="-6" x2="3" y2="-6" width="1.27" layer="1"/>
+<wire x1="3" y1="-6" x2="1.5" y2="-4.5" width="1.27" layer="1"/>
+<wire x1="82.5" y1="48" x2="82.5" y2="43.5" width="1.27" layer="1"/>
+<wire x1="63" y1="12" x2="45" y2="-6" width="1.27" layer="1"/>
 </signal>
 <signal name="S$4">
@@
 <contactref element="E$1" pad="GND"/>
 <contactref element="E$3" pad="J2.16"/>
+<wire x1="14.55" y1="0.45" x2="13.85" y2="0.45" width="1.27" layer="1"/>
+<wire x1="54.62" y1="45.88" x2="54.62" y2="46.05" width="1.27" layer="1"/>
 <wire x1="13.85" y1="0.45" x2="14.55" y2="0.45" width="1.27" layer="1"/>
 <wire x1="14.55" y1="0.45" x2="16.5" y2="-1.5" width="1.27" layer="1"/>
-<wire x1="16.5" y1="-1.5" x2="27" y2="-1.5" width="1.27" layer="1"/>
-<wire x1="27" y1="-1.5" x2="57" y2="28.5" width="1.27" layer="1"/>
-<wire x1="54.62" y1="46.05" x2="54.62" y2="45.88" width="1.27" layer="1"/>
-<wire x1="54.62" y1="45.88" x2="57" y2="43.5" width="1.27" layer="1"/>
-<wire x1="57" y1="43.5" x2="57" y2="28.5" width="1.27" layer="1"/>
+<wire x1="16.5" y1="-1.5" x2="40.5" y2="-1.5" width="1.27" layer="1"/>
+<wire x1="57" y1="15" x2="40.5" y2="-1.5" width="1.27" layer="1"/>
+<wire x1="54.62" y1="46.05" x2="54.62" y2="44.38" width="1.27" layer="1"/>
+<wire x1="54.62" y1="44.38" x2="57" y2="42" width="1.27" layer="1"/>
+<wire x1="57" y1="42" x2="57" y2="15" width="1.27" layer="1"/>
 </signal>
 <signal name="S$9">
 <contactref element="E$1" pad="5V"/>
 <contactref element="E$3" pad="J2.15"/>
-<wire x1="13.85" y1="2.99" x2="23.99" y2="2.99" width="1.27" layer="1"/>
-<wire x1="52.08" y1="46.05" x2="52.08" y2="31.08" width="1.27" layer="1"/>
-<wire x1="52.08" y1="31.08" x2="23.99" y2="2.99" width="1.27" layer="1"/>
+<wire x1="37.49" y1="2.99" x2="13.85" y2="2.99" width="1.27" layer="1"/>
+<wire x1="52.08" y1="46.05" x2="52.08" y2="17.58" width="1.27" layer="1"/>
+<wire x1="52.08" y1="17.58" x2="37.49" y2="2.99" width="1.27" layer="1"/>
+</signal>
+<signal name="S$10">
+<contactref element="E$2" pad="SS"/>
+<contactref element="E$4" pad="8"/>
+<wire x1="30" y1="23.89" x2="22.5" y2="23.89" width="1.27" layer="1"/>
+</signal>
+<signal name="S$11">
+<contactref element="E$2" pad="SCK"/>
+<contactref element="E$4" pad="7"/>
+<wire x1="22.5" y1="21.35" x2="30" y2="21.35" width="1.27" layer="1"/>
+</signal>
+<signal name="S$12">
+<contactref element="E$2" pad="MOSI"/>
+<contactref element="E$4" pad="6"/>
+<wire x1="30" y1="18.81" x2="22.5" y2="18.81" width="1.27" layer="1"/>
+</signal>
+<signal name="S$13">
+<contactref element="E$2" pad="MISO"/>
+<contactref element="E$4" pad="5"/>
+<wire x1="22.5" y1="16.27" x2="30" y2="16.27" width="1.27" layer="1"/>
+</signal>
+<signal name="S$15">
+<contactref element="E$2" pad="3V3"/>
+<wire x1="30" y1="6.11" x2="29.89" y2="6.11" width="1.27" layer="1"/>
+<contactref element="E$4" pad="1"/>
+<wire x1="22.5" y1="6.11" x2="30" y2="6.11" width="1.27" layer="1"/>
+</signal>
+<signal name="S$16">
+<contactref element="E$4" pad="2"/>
+<contactref element="E$2" pad="RST"/>
+<wire x1="30" y1="8.65" x2="22.5" y2="8.65" width="1.27" layer="1"/>
+</signal>
+<signal name="S$14">
+<contactref element="E$2" pad="IRQ"/>
+<contactref element="E$4" pad="4"/>
+<wire x1="30" y1="13.73" x2="22.5" y2="13.73" width="1.27" layer="1"/>
+</signal>
+<signal name="S$17">
+<contactref element="E$2" pad="GND"/>
+<contactref element="E$4" pad="3"/>
+<wire x1="30" y1="11.19" x2="22.5" y2="11.19" width="1.27" layer="1"/>
 </signal>
 </signals>
