File: Arduino/lock_board2.brd (EAGLE design)
At the start: 132 x 96 mm, 11 parts

Commit message: Preparing to add token
Parts:
- added E$10: (no value), con-lsta:FE05-1
- added E$11: (no value), diode:P1-12E
- added E$3: (no value), con-lsta:FE15
- E$2: device v-reg-3:317TL -> v-reg:317TL
Connections:
- new net S$1: E$1.D0, E$3.1
- new net S$11: E$1.D1, E$3.2
- new net S$12: E$1.D2, E$3.3
- new net S$13: E$1.D3, E$3.4
- new net S$14: E$1.D4, E$3.5
- new net S$15: E$1.3V3@1, E$3.6
- new net S$16: E$1.GND@2, E$3.7
- new net S$17: E$1.D5, E$3.8
- new net S$18: E$1.D6, E$3.9
- new net S$19: E$1.D7, E$3.10
- new net S$20: E$1.RX, E$3.12
- new net S$21: E$1.TX, E$3.13
- new net S$24: E$1.3V3@2, E$3.15
- new net S$25: E$1.GND@3, E$3.14
- net S$10: now also E$10.5
- net S$4: now also E$3.11
- net S$5: now also E$11.C
- net S$7: now also E$11.A
Routing:
- net S$10: track 7.49 -> 18.2 mm
- net S$7: track 143.5 -> 151.4 mm
- net S$5: track 11.1 -> 17.4 mm
- net S$4: track 80.6 -> 85.9 mm
- net S$25: track 0.00 -> 5.33 mm
- net S$24: track 0.00 -> 5.33 mm
- net S$20: track 0.00 -> 5.33 mm
- net S$19: track 0.00 -> 5.33 mm
- net S$12: track 0.00 -> 5.33 mm
- net S$11: track 0.00 -> 5.33 mm
- net S$18: track 0.00 -> 5.33 mm
- net S$17: track 0.00 -> 5.33 mm
- net S$16: track 0.00 -> 5.33 mm
- net S$15: track 0.00 -> 5.33 mm
- net S$14: track 0.00 -> 5.33 mm
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Other:
- board outline removed
- board text removed: "GND"
- board text removed: "VCC"
- board text removed: "lock"
- board text removed: "power supply"

Commit message: code with token
Connections:
- net S$10: now also E$10.1, E$10.2, E$10.3, E$10.4
Routing:
- net S$10: track 18.2 -> 28.3 mm
Changed lines of the file:
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@@
 <wire x1="47.08" y1="82.5" x2="47.08" y2="72.54" width="1.27" layer="1"/>
 <wire x1="47.08" y1="72.54" x2="47.58" y2="72.04" width="1.27" layer="1"/>
+<contactref element="E$10" pad="4"/>
+<contactref element="E$10" pad="3"/>
+<contactref element="E$10" pad="2"/>
+<contactref element="E$10" pad="1"/>
+<wire x1="36.92" y1="82.5" x2="47.08" y2="82.5" width="1.27" layer="1"/>
+<wire x1="42" y1="82.5" x2="44.54" y2="82.5" width="0" layer="19" extent="1-1"/>
+<wire x1="39.46" y1="82.5" x2="42" y2="82.5" width="0" layer="19" extent="1-1"/>
+<wire x1="47.08" y1="82.5" x2="44.54" y2="82.5" width="0" layer="19" extent="1-1"/>
 </signal>
 <signal name="S$22">
