File: Arduino/PlatformIO/antena_regulador.brd (EAGLE design)
At the start: 7 parts

Commit message: Deleted .b#* files
Parts:
- removed E$6, E$7: (no value), con-lstb:MA03-1
- E$4: device con-lstb:MA03-1 -> con-lstb:MA04-1
- moved E$4 1.19 mm to (88.6, 54.0), turned to 90 degrees
Connections:
- removed net S$5: E$2.2, E$4.2, E$5.2, E$6.2, E$7.2
- new net S$2: E$1.2, E$3.1, E$4.2
- net S$3: now also E$2.2, E$4.3, E$5.2; no longer E$1.3, E$5.1
- net S$4: now also E$1.3, E$4.4, E$5.1; no longer E$1.2, E$3.1, E$6.1, E$7.1
Routing:
- net S$5: track 42.8 -> 0.00 mm
- net S$2: track 0.00 -> 34.5 mm
- net S$3: track 31.4 -> 38.4 mm
- net S$4: track 35.2 -> 32.1 mm
Changed lines of the file:
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@@
 <element name="E$2" library="eagle-ltspice" package="0207/10" value="" x="74.93" y="31.75"/>
 <element name="E$3" library="eagle-ltspice" package="0207/10" value="" x="74.93" y="36.83" rot="R180"/>
+<element name="E$4" library="con-lstb" package="MA04-1" value="" x="88.63" y="53.99" rot="R90"/>
 <element name="E$5" library="con-lstb" package="MA03-1" value="" x="96" y="55" rot="R270"/>
-<element name="E$4" library="con-lstb" package="MA03-1" value="" x="88" y="55" rot="R270"/>
-<element name="E$6" library="con-lstb" package="MA03-1" value="" x="88" y="47" rot="R270"/>
-<element name="E$7" library="con-lstb" package="MA03-1" value="" x="88" y="39" rot="R270"/>
 </elements>
 <signals>
@@
 <wire x1="69.85" y1="31.75" x2="69.85" y2="36.83" width="1.4224" layer="1"/>
 </signal>
-<signal name="S$5">
-<contactref element="E$5" pad="2"/>
-<wire x1="96" y1="55.26" x2="96" y2="55" width="1.27" layer="1"/>
-<wire x1="96" y1="55.26" x2="95.74" y2="55" width="1.27" layer="1"/>
-<contactref element="E$4" pad="2"/>
-<contactref element="E$2" pad="2"/>
-<contactref element="E$6" pad="2"/>
-<contactref element="E$7" pad="2"/>
-<wire x1="88" y1="39" x2="90" y2="39" width="1.27" layer="1"/>
-<wire x1="90" y1="39" x2="91" y2="40" width="1.27" layer="1"/>
-<wire x1="91" y1="40" x2="91" y2="46" width="1.27" layer="1"/>
-<wire x1="91" y1="46" x2="90" y2="47" width="1.27" layer="1"/>
-<wire x1="88" y1="47" x2="90" y2="47" width="1.27" layer="1"/>
-<wire x1="90" y1="47" x2="91" y2="48" width="1.27" layer="1"/>
-<wire x1="91" y1="48" x2="91" y2="54" width="1.27" layer="1"/>
-<wire x1="88" y1="55" x2="90" y2="55" width="1.27" layer="1"/>
-<wire x1="90" y1="55" x2="91" y2="54" width="1.27" layer="1"/>
-<wire x1="95.74" y1="55" x2="92" y2="55" width="1.27" layer="1"/>
-<wire x1="92" y1="55" x2="91" y2="54" width="1.27" layer="1"/>
-<wire x1="80.01" y1="31.75" x2="82.75" y2="31.75" width="1.27" layer="1"/>
-<wire x1="82.75" y1="31.75" x2="84" y2="33" width="1.27" layer="1"/>
-<wire x1="84" y1="33" x2="84" y2="37" width="1.27" layer="1"/>
-<wire x1="88" y1="39" x2="86" y2="39" width="1.27" layer="1"/>
-<wire x1="86" y1="39" x2="84" y2="37" width="1.27" layer="1"/>
-</signal>
-<signal name="S$3">
-<contactref element="E$4" pad="1"/>
-<contactref element="E$1" pad="3"/>
-<contactref element="E$5" pad="1"/>
-<wire x1="96" y1="57.8" x2="96" y2="57.54" width="1.27" layer="1"/>
-<wire x1="74.93" y1="43.18" x2="77.18" y2="43.18" width="1.27" layer="1"/>
-<wire x1="77.18" y1="43.18" x2="80" y2="46" width="1.27" layer="1"/>
-<wire x1="80" y1="46" x2="80" y2="53" width="1.27" layer="1"/>
-<wire x1="80" y1="53" x2="84.54" y2="57.54" width="1.27" layer="1"/>
-<wire x1="88" y1="57.54" x2="84.54" y2="57.54" width="1.27" layer="1"/>
-<wire x1="96" y1="57.54" x2="88" y2="57.54" width="1.27" layer="1"/>
-</signal>
-<signal name="S$4">
-<contactref element="E$7" pad="1"/>
-<contactref element="E$6" pad="1"/>
+<signal name="S$2">
 <contactref element="E$1" pad="2"/>
 <contactref element="E$3" pad="1"/>
@@
 <wire x1="79" y1="40" x2="80" y2="39" width="1.4224" layer="1"/>
 <wire x1="80" y1="39" x2="80" y2="37" width="1.4224" layer="1"/>
+<contactref element="E$4" pad="2"/>
+<wire x1="88.63" y1="52.72" x2="86.72" y2="52.72" width="1.4224" layer="1"/>
+<wire x1="86.72" y1="52.72" x2="85" y2="51" width="1.4224" layer="1"/>
+<wire x1="85" y1="51" x2="85" y2="40" width="1.4224" layer="1"/>
+<wire x1="85" y1="40" x2="82" y2="37" width="1.4224" layer="1"/>
+<wire x1="82" y1="37" x2="80.18" y2="37" width="1.4224" layer="1"/>
 <wire x1="80.18" y1="37" x2="80.01" y2="36.83" width="1.4224" layer="1"/>
-<wire x1="88" y1="49.54" x2="85.54" y2="49.54" width="1.27" layer="1"/>
-<wire x1="85.54" y1="49.54" x2="84" y2="48" width="1.27" layer="1"/>
-<wire x1="84" y1="48" x2="84" y2="43" width="1.27" layer="1"/>
-<wire x1="84" y1="43" x2="85.46" y2="41.54" width="1.27" layer="1"/>
-<wire x1="88" y1="41.54" x2="85.46" y2="41.54" width="1.27" layer="1"/>
-<wire x1="80.01" y1="36.83" x2="80.01" y2="39.01" width="1.27" layer="1"/>
-<wire x1="80.01" y1="39.01" x2="84" y2="43" width="1.27" layer="1"/>
-<wire x1="80" y1="39" x2="80.01" y2="39.01" width="0" layer="19" extent="1-1"/>
+<wire x1="80" y1="37" x2="80.01" y2="36.83" width="0" layer="19" extent="1-1"/>
+</signal>
+<signal name="S$3">
+<contactref element="E$2" pad="2"/>
+<contactref element="E$4" pad="1"/>
+<wire x1="80.01" y1="31.75" x2="81.75" y2="31.75" width="1.4224" layer="1"/>
+<wire x1="81.75" y1="31.75" x2="88.63" y2="38.63" width="1.4224" layer="1"/>
+<wire x1="88.63" y1="50.18" x2="88.63" y2="38.63" width="1.4224" layer="1"/>
+<contactref element="E$4" pad="3"/>
+<wire x1="88.63" y1="50.18" x2="91.18" y2="50.18" width="1.4224" layer="1"/>
+<wire x1="91.18" y1="50.18" x2="92" y2="51" width="1.4224" layer="1"/>
+<wire x1="88.63" y1="55.26" x2="90.74" y2="55.26" width="1.4224" layer="1"/>
+<wire x1="90.74" y1="55.26" x2="92" y2="54" width="1.4224" layer="1"/>
+<wire x1="92" y1="54" x2="92" y2="51" width="1.4224" layer="1"/>
+<contactref element="E$5" pad="2"/>
+<wire x1="96" y1="55.26" x2="96" y2="55" width="1.27" layer="1"/>
+<wire x1="96" y1="55.26" x2="95.74" y2="55" width="1.27" layer="1"/>
+<wire x1="95.74" y1="55" x2="93" y2="55" width="1.27" layer="1"/>
+<wire x1="92" y1="54" x2="93" y2="55" width="1.27" layer="1"/>
+</signal>
+<signal name="S$4">
+<contactref element="E$4" pad="4"/>
+<contactref element="E$1" pad="3"/>
+<wire x1="74.93" y1="43.18" x2="79.18" y2="43.18" width="1.4224" layer="1"/>
+<wire x1="79.18" y1="43.18" x2="81" y2="45" width="1.4224" layer="1"/>
+<wire x1="88.63" y1="57.8" x2="85.8" y2="57.8" width="1.4224" layer="1"/>
+<wire x1="85.8" y1="57.8" x2="81" y2="53" width="1.4224" layer="1"/>
+<wire x1="81" y1="53" x2="81" y2="45" width="1.4224" layer="1"/>
+<contactref element="E$5" pad="1"/>
+<wire x1="88.63" y1="57.8" x2="96" y2="57.8" width="1.27" layer="1"/>
+<wire x1="96" y1="57.8" x2="96" y2="57.54" width="1.27" layer="1"/>
 </signal>
 </signals>
