File: Arduino/Placas/sirene.brd (EAGLE design)
At the start: 9 parts

Commit message: Sirene board updated
Parts:
- removed E$7: (no value), con-lstb:MA03-1
- E$6: device jumper:0R/10 -> con-lstb:MA04-1
- moved E$4 24.6 mm to (33.9, 45.5)
- moved 720 21.1 mm to (45.6, 46.5)
- moved 220 17.1 mm to (45.6, 52.4)
- moved E$3 15.7 mm to (33.9, 57.5)
- moved E$2 14.2 mm to (47.0, 64.9)
- moved E$5 5.41 mm to (37.5, 28.5), turned to 0 degrees
- moved E$6 4.50 mm to (48.0, 33.0), turned to 270 degrees
Connections:
- removed net S$6: E$1.D1, E$6.2
- new net S$4: E$1.3V3@2, E$6.3
- new net S$9: E$4.2, E$5.2
- net S$1: now also E$5.1; no longer E$7.2
- net S$2: no longer E$5.1
- net S$5: now also E$1.D1; no longer E$5.3
- net S$7: now also E$6.2; no longer E$4.2, E$5.2, E$7.3
Routing:
- net S$2: track 166.3 -> 48.1 mm
- net S$7: track 179.2 -> 112.7 mm
- net S$4: track 0.00 -> 55.3 mm
- net S$1: track 92.6 -> 58.4 mm
- net S$9: track 0.00 -> 24.5 mm
- net S$6: track 8.17 -> 0.00 mm
- net S$5: track 7.47 -> 13.8 mm
- net S$3: track 15.2 -> 20.8 mm
Other:
- board outline added: 57 x 51 mm
- board text added: "+"
- board text added: "220"
- board text added: "680"
- board text added: "IN"
- board text added: "SIR"

Commit message: Sirene board updated
Parts:
- removed 220, 720: (no value), rcl:0207/7
- removed E$2: (no value), v-reg:317TL
- removed E$3, E$4: (no value), con-weidmueller-sl35:180G-2
- removed E$5: (no value), con-lstb:MA03-1
- removed E$6: (no value), con-lstb:MA04-1
- added 21, 22: (no value), rcl:0207/7
- added E$68: (no value), v-reg:317TL
- added E$69, E$70: (no value), con-weidmueller-sl35:180G-2
- added E$71: (no value), con-lstb:MA04-1
- added E$72: (no value), con-lstb:MA03-1
- E$1: device ESP12E_DEVKIT:ESP12E_DEVKIT -> Lolin:LOLIN
- moved E$1 167.9 mm to (-48.0, 166.5), turned to 90 degrees
Connections:
- removed net S$1: E$2.3, E$3.2, E$5.1
- removed net S$2: 220.1, E$1.VIN, E$2.2
- removed net S$3: 220.2, 720.1, E$2.1
- removed net S$4: E$1.3V3@2, E$6.3
- removed net S$5: E$1.D1, E$6.1
- removed net S$7: 720.2, E$1.GND@1, E$3.1, E$4.1, E$6.2
- removed net S$9: E$4.2, E$5.2
- new net S$80: E$68.3, E$69.2, E$72.1
- new net S$81: 22.1, E$1.VIN, E$68.2
- new net S$82: 21.1, 22.2, E$68.1
- new net S$83: E$70.2, E$72.2
- new net S$84: E$1.3V1, E$71.3
- new net S$85: E$1.D1, E$71.1
- new net S$86: 21.2, E$1.G2, E$69.1, E$70.1, E$71.2
Routing:
- net S$86: track 0.00 -> 116.9 mm
- net S$7: track 112.7 -> 0.00 mm
- net S$80: track 0.00 -> 58.4 mm
- net S$1: track 58.4 -> 0.00 mm
- net S$4: track 55.3 -> 0.00 mm
- net S$84: track 0.00 -> 55.2 mm
- net S$81: track 0.00 -> 53.0 mm
- net S$2: track 48.1 -> 0.00 mm
- net S$83: track 0.00 -> 24.5 mm
- net S$9: track 24.5 -> 0.00 mm
- net S$3: track 20.8 -> 0.00 mm
- net S$82: track 0.00 -> 20.8 mm
- net S$85: track 0.00 -> 14.4 mm
- net S$5: track 13.8 -> 0.00 mm
Other:
- board size 57 x 51 mm -> 30.5 x 47.6 mm

Commit message: Finished sirene board project
Parts:
- added 1, 10, 11, 12, 13, 14, 2, 3, 4, 5, 6, 7, 8, 9: (no value), rcl:0207/7
- added E$10, E$15, E$16, E$21, E$22, E$27, E$28, E$3, E$33, E$34, E$39, E$4, E$40, E$9: (no value), con-weidmueller-sl35:180G-2
- added E$11, E$17, E$23, E$29, E$35, E$41, E$5: (no value), con-lstb:MA04-1
- added E$12, E$18, E$24, E$30, E$36, E$42, E$6: (no value), con-lstb:MA03-1
- added E$13, E$19, E$25, E$31, E$37, E$43, E$7: (no value), Lolin:LOLIN
- added E$14, E$2, E$20, E$26, E$32, E$38, E$8: (no value), v-reg:317TL
- moved E$69 40.2 mm to (-80.0, 138.9), turned to 180 degrees
- moved E$68 38.6 mm to (-87.4, 152.0), turned to 90 degrees
- moved E$70 31.9 mm to (-68.0, 138.9), turned to 180 degrees
- moved E$72 29.5 mm to (-51.0, 142.5), turned to 90 degrees
- moved 22 23.5 mm to (-74.9, 150.6), turned to 270 degrees
- moved E$1 20.9 mm to (-67.5, 174.0), turned to 180 degrees
- moved 21 17.5 mm to (-69.0, 150.6), turned to 270 degrees
- moved E$71 13.6 mm to (-55.5, 153.0), turned to 0 degrees
Connections:
- new net S$1: E$2.3, E$3.2, E$6.1
- new net S$11: 4.1, E$13.VIN, E$8.2
- new net S$12: 3.1, 4.2, E$8.1
- new net S$13: E$10.2, E$12.2
- new net S$14: E$11.3, E$13.3V1
- new net S$15: E$11.1, E$13.D1
- new net S$16: 3.2, E$10.1, E$11.2, E$13.G2, E$9.1
- new net S$17: E$14.3, E$15.2, E$18.1
- new net S$18: 6.1, E$14.2, E$19.VIN
- new net S$19: 5.1, 6.2, E$14.1
- new net S$2: 2.1, E$2.2, E$7.VIN
- new net S$20: E$16.2, E$18.2
- new net S$21: E$17.3, E$19.3V1
- new net S$22: E$17.1, E$19.D1
- new net S$23: 5.2, E$15.1, E$16.1, E$17.2, E$19.G2
- new net S$24: E$20.3, E$21.2, E$24.1
- new net S$25: 8.1, E$20.2, E$25.VIN
- new net S$26: 7.1, 8.2, E$20.1
- new net S$27: E$22.2, E$24.2
- new net S$28: E$23.3, E$25.3V1
- new net S$29: E$23.1, E$25.D1
- new net S$3: 1.1, 2.2, E$2.1
- new net S$30: 7.2, E$21.1, E$22.1, E$23.2, E$25.G2
- new net S$31: E$26.3, E$27.2, E$30.1
- new net S$32: 10.1, E$26.2, E$31.VIN
- new net S$33: 10.2, 9.1, E$26.1
- new net S$34: E$28.2, E$30.2
- new net S$35: E$29.3, E$31.3V1
- new net S$36: E$29.1, E$31.D1
- new net S$37: 9.2, E$27.1, E$28.1, E$29.2, E$31.G2
- new net S$38: E$32.3, E$33.2, E$36.1
- new net S$39: 12.1, E$32.2, E$37.VIN
- new net S$4: E$4.2, E$6.2
- new net S$40: 11.1, 12.2, E$32.1
- new net S$41: E$34.2, E$36.2
- new net S$42: E$35.3, E$37.3V1
- new net S$43: E$35.1, E$37.D1
- new net S$44: 11.2, E$33.1, E$34.1, E$35.2, E$37.G2
- new net S$45: E$38.3, E$39.2, E$42.1
- new net S$46: 14.1, E$38.2, E$43.VIN
- new net S$47: 13.1, 14.2, E$38.1
- new net S$48: E$40.2, E$42.2
- new net S$49: E$41.3, E$43.3V1
- new net S$5: E$5.3, E$7.3V1
- new net S$50: E$41.1, E$43.D1
- new net S$51: 13.2, E$39.1, E$40.1, E$41.2, E$43.G2
- new net S$7: E$5.1, E$7.D1
- new net S$8: 1.2, E$3.1, E$4.1, E$5.2, E$7.G2
- new net S$9: E$12.1, E$8.3, E$9.2
Routing:
- net S$37: track 0.00 -> 116.9 mm
- net S$51: track 0.00 -> 116.9 mm
- net S$44: track 0.00 -> 116.9 mm
- net S$30: track 0.00 -> 116.9 mm
- net S$8: track 0.00 -> 116.9 mm
- net S$23: track 0.00 -> 116.9 mm
- net S$16: track 0.00 -> 116.9 mm
- net S$38: track 0.00 -> 58.4 mm
- net S$9: track 0.00 -> 58.4 mm
- net S$45: track 0.00 -> 58.4 mm
- net S$24: track 0.00 -> 58.4 mm
- net S$1: track 0.00 -> 58.4 mm
- net S$17: track 0.00 -> 58.4 mm
- net S$31: track 0.00 -> 58.4 mm
- net S$28: track 0.00 -> 55.2 mm
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Other:
- board size 30.5 x 47.6 mm -> 47.6 x 30.5 mm
