File: Placas/lock-board_lock_v3.brd (EAGLE design)
At the start: 23 parts

Commit message: Finished project, needs testing and refactoring
Parts:
- removed E$14, E$16, E$8: (no value), con-lstb:MA03-1
Connections:
- net S$46: no longer E$14.2, E$8.2
- net S$68: no longer E$16.2
- net S$73: no longer E$14.1, E$16.1, E$8.1
Routing:
- net S$73: track 192.9 -> 159.1 mm
- net S$46: track 134.8 -> 107.6 mm
- net S$68: track 101.9 -> 108.6 mm
Other:
- board text added: "+ -"
- board text removed: "- +"
- board text removed: "ANT1"
- board text removed: "ANT2"
- board text removed: "US"
